File: Zeichenmaschine/Zeichenmaschine.kicad_sch (KiCad schematic)
At the start: 37 parts, among them J1 interface_panel_0, J10 Conn_01x02_Male, J11 USB_C, J12 Conn_01x02_Male, J13 interface_panel_1, J2 Stepper_1, J3 Stepper_2, J4 Screw_Terminal_01x02, J5 Display, J6 Stepper_2_JUMPER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

Commit message: test2
Parts:
- added A3: Stepper_2_A4988, Module:Pololu_Breakout-16_15.2x20.3mm, symbol Driver_Motor:Pololu_Breakout_A4988
- added J14: Stepper_3_JUMPER, Connector_PinHeader_2.54mm:PinHeader_2x03_P2.54mm_Vertical, symbol Connector:Conn_01x06_Male
- added J15: Stepper_2, Connector_JST:JST_EH_B4B-EH-A_1x04_P2.50mm_Vertical, symbol Connector:Conn_01x04_Male
Connections:
- net +12V: now also A3.8 (VMOT)
- net +5V: now also A3.2 (VDD), J14.1 (Pin_1), J14.3 (Pin_3), J14.5 (Pin_5)
- net GND: now also A3.1 (GND), A3.7 (GND)
- net dc_gear_motor_1A: now also A3.15 (STEP)
- net dc_gear_motor_2A: now also A3.16 (DIR)
- net enable_dc_gear_motor: now also A3.9 (~{ENABLE})
- new net: A3.10 (MS1), J14.2 (Pin_2)
- new net: A3.11 (MS2), J14.4 (Pin_4)
- new net: A3.12 (MS3), J14.6 (Pin_6)
- new net: A3.13 (~{RESET}), A3.14 (~{SLEEP})
- new net: A3.3 (1B), J15.4 (Pin_4)
- new net: A3.4 (1A), J15.3 (Pin_3)
- new net: A3.5 (2A), J15.2 (Pin_2)
- new net: A3.6 (2B), J15.1 (Pin_1)
- no-connect marks 20 -> 21
Other:
- moved on the sheet: A2, J3, J5, J6, J7, J9

Commit message: asjhgdnsa
Parts:
- removed J13: interface_panel_1, Connector_JST:JST_EH_B5B-EH-A_1x05_P2.50mm_Vertical, symbol Connector:Conn_01x05_Male
- added D5: D_Schottky, Diode_THT:D_5W_P12.70mm_Horizontal, symbol Device:D_Schottky
- added R5: 1k, Resistor_THT:R_Axial_DIN0204_L3.6mm_D1.6mm_P7.62mm_Horizontal, symbol Device:R
- added R6: 270, Resistor_THT:R_Axial_DIN0204_L3.6mm_D1.6mm_P7.62mm_Horizontal, symbol Device:R
- A3: value Stepper_2_A4988 -> Stepper_3_A4988
- J1: value interface_panel_0 -> interface
- J15: value Stepper_2 -> Stepper_3
Connections:
- net +12V: now also D5.1 (K); no longer J4.2 (Pin_2)
- net +5V: now also J1.5 (Pin_5)
- net GND: now also R5.2, R6.2; no longer J1.1 (Pin_1)
- net at A3.3 (1B): now also J15.1 (Pin_1); no longer J15.4 (Pin_4)
- net at A3.4 (1A): now also J15.2 (Pin_2); no longer J15.3 (Pin_3)
- net at A3.5 (2A): now also J15.3 (Pin_3); no longer J15.2 (Pin_2)
- net at A3.6 (2B): now also J15.4 (Pin_4); no longer J15.1 (Pin_1)
- net at A1.3 (1B): now also J2.1 (Pin_1); no longer J2.4 (Pin_4)
- net at A1.4 (1A): now also J2.2 (Pin_2); no longer J2.3 (Pin_3)
- net at A1.5 (2A): now also J2.3 (Pin_3); no longer J2.2 (Pin_2)
- net at A1.6 (2B): now also J2.4 (Pin_4); no longer J2.1 (Pin_1)
- net at A2.3 (1B): now also J3.1 (Pin_1); no longer J3.4 (Pin_4)
- net at A2.4 (1A): now also J3.2 (Pin_2); no longer J3.3 (Pin_3)
- net at A2.5 (2A): now also J3.3 (Pin_3); no longer J3.2 (Pin_2)
- net at A2.6 (2B): now also J3.4 (Pin_4); no longer J3.1 (Pin_1)
- net interface_btn: now reaches U4.10 (DAC_2/ADC2_CH9/GPIO26)
- net interface_btn: now also J1.1 (Pin_1), R5.1
- net interface_poti: now reaches U4.9 (DAC_1/ADC2_CH8/GPIO25)
- net interface_poti: now also J1.4 (Pin_4)
- net DN: no longer names the net of U4.4 (SENSOR_VN/GPIO39/ADC1_CH3)
- net DN: no longer J1.4 (Pin_4)
- net MN: no longer names the net of U4.7 (32K_XP/GPIO32/ADC1_CH4)
- net PW: no longer names the net of U4.5 (VDET_1/GPIO34/ADC1_CH6)
- net PW: no longer J1.5 (Pin_5)
- net SEL: no longer names the net of U4.6 (VDET_2/GPIO35/ADC1_CH7)
- net UP: no longer names the net of J1.3 (Pin_3)
- net UP: now also R6.1; no longer U4.3 (SENSOR_VP/GPIO36/ADC1_CH0)
- new net: D5.2 (A), J4.2 (Pin_2)
- no-connect marks 21 -> 23
Other:
- moved on the sheet: J1, J15, J2, J3
